Commit message: changed namespace to komodo_1

File: ric/ric_description/komodo/komodo.xacro (robot description, xacro)
@@ -1,6 +1,25 @@
 <?xml version="1.0"?>
-<robot xmlns:xacro="http://www.ros.org/wiki/ric" name="ric_description">
-  <link
-    name="komodo_$(arg komodo_id)_base_link">
+<robot
+  name="komodo_$(arg komodo_id)">
+<!-- Dummy inertia link & Joint -->
+  <link
+    name="dummy_link">
+</link>
+  <joint
+    name="dummy_joint"
+    type="fixed">
+    <origin
+      xyz="0.0 0.0 0.0"
+      rpy="0 0 0" />
+    <parent
+      link="dummy_link" />
+    <child
+      link="base_link" />
+    <axis
+      xyz="0 0 0" />
+  </joint>
+<!-- Dummy link & node -->
+  <link
+    name="base_link">
     <inertial>
       <origin
@@ -8,20 +27,20 @@
         rpy="0 0 0" />
       <mass
-        value="4.50894999160313" />
-      <inertia
-        ixx="0.0723503030508731"
-        ixy="-4.68485359152423E-05"
-        ixz="-0.00875564429068847"
-        iyy="0.138127064231828"
-        iyz="1.19695110167269E-05"
-        izz="0.194371448739423" />
-    </inertial>
-    <visual>
-      <origin
-        xyz="0 0 0"
-        rpy="0 0 0" />
-      <geometry>
-        <mesh
-          filename="package://ric_description/komodo/meshes/base_link.STL" />
+        value="45.0894999160313" />
+      <inertia
+        ixx="0.723503030508731"
+        ixy="-46.8485359152423E-05"
+        ixz="-0.0875564429068847"
+        iyy="1.38127064231828"
+        iyz="11.9695110167269E-05"
+        izz="1.94371448739423" />
+    </inertial>
+    <visual>
+      <origin
+        xyz="0 0 0"
+        rpy="0 0 0" />
+      <geometry>
+        <mesh
+          filename="package://ric_description/komodo/meshes/col_base_link.STL" />
       </geometry>
       <material
@@ -33,14 +52,14 @@
     <collision>
       <origin
-        xyz="0 0 0"
-        rpy="0 0 0" />
-      <geometry>
-        <mesh
-          filename="package://ric_description/komodo/meshes/base_link.STL" />
-      </geometry>
-    </collision>
-  </link>
-  <link
-    name="komodo_$(arg komodo_id)_FR_Wheel_link">
+        xyz="-0.065 0 0"
+        rpy="0 0 0" />
+      <geometry>
+        <mesh
+          filename="package://ric_description/komodo/meshes/col_base_link.STL" />
+      </geometry>
+    </collision>
+  </link>
+  <link
+    name="FR_Wheel_link">
     <inertial>
       <origin
@@ -74,26 +93,28 @@
       <origin
         xyz="0 0 0"
-        rpy="0 0 0" />
-      <geometry>
-        <mesh
-          filename="package://ric_description/komodo/meshes/FR_Wheel_link.STL" />
-      </geometry>
-    </collision>
-  </link>
-  <joint
-    name="komodo_$(arg komodo_id)_FR_Wheel_joint"
+        rpy="0 1.5 0" />
+      <geometry>
+       <!--mesh
+          filename="package://ric_description/komodo/meshes_elevator/FR_Wheel_link.STL" /-->
+        <cylinder length="0.05" radius="0.1"
+          />
+      </geometry>
+    </collision>
+  </link>
+  <joint
+    name="FR_Wheel_joint"
     type="continuous">
     <origin
       xyz="0.173999999999995 -0.2009 0"
-      rpy="2.62229105359916E-15 6.9308460464278E-17 -1.5707963267949" />
-    <parent
-      link="komodo_$(arg komodo_id)_base_link" />
-    <child
-      link="komodo_$(arg komodo_id)_FR_Wheel_link" />
+      rpy="2.62229105359916E-15 6.9308460464278E-17 1.5707963267949" />
+    <parent
+      link="base_link" />
+    <child
+      link="FR_Wheel_link" />
     <axis
       xyz="1 0 0" />
   </joint>
   <link
-    name="komodo_$(arg komodo_id)_FL_Wheel_link">
+    name="FL_Wheel_link">
     <inertial>
       <origin
@@ -127,26 +148,28 @@
       <origin
         xyz="0 0 0"
-        rpy="0 0 0" />
-      <geometry>
-        <mesh
-          filename="package://ric_description/komodo/meshes/FL_Wheel_link.STL" />
-      </geometry>
-    </collision>
-  </link>
-  <joint
-    name="komodo_$(arg komodo_id)_FL_Wheel_joint"
+        rpy="0 1.5 0" />
+      <geometry>
+       <!--mesh
+          filename="package://ric_description/komodo/meshes_elevator/FR_Wheel_link.STL" /-->
+        <cylinder length="0.05" radius="0.1"
+          />
+      </geometry>
+    </collision>
+  </link>
+  <joint
+    name="FL_Wheel_joint"
     type="continuous">
     <origin
       xyz="0.173999999999995 0.2009 0"
-      rpy="-2.62229105359916E-15 6.93084604642783E-17 1.5707963267949" />
-    <parent
-      link="komodo_$(arg komodo_id)_base_link" />
-    <child
-      link="komodo_$(arg komodo_id)_FL_Wheel_link" />
+      rpy="-2.62229105359916E-15 6.93084604642783E-17 -1.5707963267949" />
+    <parent
+      link="base_link" />
+    <child
+      link="FL_Wheel_link" />
     <axis
       xyz="-1 0 0" />
   </joint>
   <link
-    name="komodo_$(arg komodo_id)_RR_Wheel_link">
+    name="RR_Wheel_link">
     <inertial>
       <origin
@@ -180,26 +203,28 @@
       <origin
         xyz="0 0 0"
-        rpy="0 0 0" />
-      <geometry>
-        <mesh
-          filename="package://ric_description/komodo/meshes/RR_Wheel_link.STL" />
-      </geometry>
-    </collision>
-  </link>
-  <joint
-    name="komodo_$(arg komodo_id)_RR_Wheel_joint"
+        rpy="0 1.5 0" />
+      <geometry>
+       <!--mesh
+          filename="package://ric_description/komodo/meshes_elevator/FR_Wheel_link.STL" /-->
+        <cylinder length="0.05" radius="0.1"
+          />
+      </geometry>
+    </collision>
+  </link>
+  <joint
+    name="RR_Wheel_joint"
     type="continuous">
     <origin
       xyz="-0.156000000000005 -0.2009 0"
-      rpy="2.62229105359916E-15 -1.59433090848306E-31 -1.5707963267949" />
-    <parent
-      link="komodo_$(arg komodo_id)_base_link" />
-    <child
-      link="komodo_$(arg komodo_id)_RR_Wheel_link" />
+      rpy="2.62229105359916E-15 -1.59433090848306E-31 1.5707963267949" />
+    <parent
+      link="base_link" />
+    <child
+      link="RR_Wheel_link" />
     <axis
       xyz="1 0 0" />
   </joint>
   <link
-    name="komodo_$(arg komodo_id)_RL_Wheel_link">
+    name="RL_Wheel_link">
     <inertial>
       <origin
@@ -233,26 +258,28 @@
       <origin
         xyz="0 0 0"
-        rpy="0 0 0" />
-      <geometry>
-        <mesh
-          filename="package://ric_description/komodo/meshes/RL_Wheel_link.STL" />
-      </geometry>
-    </collision>
-  </link>
-  <joint
-    name="komodo_$(arg komodo_id)_RL_Wheel_joint"
+        rpy="0 1.5 0" />
+      <geometry>
+       <!--mesh
+          filename="package://ric_description/komodo/meshes_elevator/FR_Wheel_link.STL" /-->
+        <cylinder length="0.05" radius="0.1"
+          />
+      </geometry>
+    </collision>
+  </link>
+  <joint
+    name="RL_Wheel_joint"
     type="continuous">
     <origin
       xyz="-0.156000000000005 0.2009 0"
-      rpy="-2.62229105359916E-15 -5.57680208627196E-32 1.5707963267949" />
-    <parent
-      link="komodo_$(arg komodo_id)_base_link" />
-    <child
-      link="komodo_$(arg komodo_id)_RL_Wheel_link" />
+      rpy="-2.62229105359916E-15 -5.57680208627196E-32 -1.5707963267949" />
+    <parent
+      link="base_link" />
+    <child
+      link="RL_Wheel_link" />
     <axis
       xyz="-1 0 0" />
   </joint>
   <link
-    name="komodo_$(arg komodo_id)_Left_URF_link">
+    name="Left_URF_link">
     <inertial>
       <origin
@@ -280,5 +307,5 @@
         name="">
         <color
-          rgba="0.1 0.1 0.1 1" />
+          rgba="0.752941176470588 0.752941176470588 0.752941176470588 1" />
       </material>
     </visual>
@@ -294,5 +321,5 @@
   </link>
   <joint
-    name="komodo_$(arg komodo_id)_Left_URF_joint"
+    name="Left_URF_joint"
     type="fixed">
     <origin
@@ -300,12 +327,12 @@
       rpy="-2.73331335606168E-15 1.59433090848306E-31 1.5707963267949" />
     <parent
-      link="komodo_$(arg komodo_id)_base_link" />
-    <child
-      link="komodo_$(arg komodo_id)_Left_URF_link" />
+      link="base_link" />
+    <child
+      link="Left_URF_link" />
     <axis
       xyz="-1 0 0" />
   </joint>
   <link
-    name="komodo_$(arg komodo_id)_Rear_URF_link">
+    name="Rear_URF_link">
     <inertial>
       <origin
@@ -333,5 +360,5 @@
         name="">
         <color
-          rgba="0.1 0.1 0.1 1" />
+          rgba="0.752941176470588 0.752941176470588 0.752941176470588 1" />
       </material>
     </visual>
@@ -347,5 +374,5 @@
   </link>
   <joint
-    name="komodo_$(arg komodo_id)_Rear_URF_joint"
+    name="Rear_URF_joint"
     type="fixed">
     <origin
@@ -353,12 +380,12 @@
       rpy="-6.16297582203915E-33 2.73331335606168E-15 3.14159265358979" />
     <parent
-      link="komodo_$(arg komodo_id)_base_link" />
-    <child
-      link="komodo_$(arg komodo_id)_Rear_URF_link" />
+      link="base_link" />
+    <child
+      link="Rear_URF_link" />
     <axis
       xyz="-1 0 0" />
   </joint>
   <link
-    name="komodo_$(arg komodo_id)_Right_URF_link">
+    name="Right_URF_link">
     <inertial>
       <origin
@@ -386,5 +413,5 @@
         name="">
         <color
-          rgba="0.1 0.1 0.1 1" />
+          rgba="0.752941176470588 0.752941176470588 0.752941176470588 1" />
       </material>
     </visual>
@@ -400,5 +427,5 @@
   </link>
   <joint
-    name="komodo_$(arg komodo_id)_Right_URF_joint"
+    name="Right_URF_joint"
     type="fixed">
     <origin
@@ -406,12 +433,12 @@
       rpy="2.73331335606168E-15 -1.59433090848306E-31 -1.5707963267949" />
     <parent
-      link="komodo_$(arg komodo_id)_base_link" />
-    <child
-      link="komodo_$(arg komodo_id)_Right_URF_link" />
+      link="base_link" />
+    <child
+      link="Right_URF_link" />
     <axis
       xyz="-1 0 0" />
   </joint>
   <link
-    name="komodo_$(arg komodo_id)_Front_Camera_link">
+    name="Front_Camera_link">
     <inertial>
       <origin
@@ -431,5 +458,5 @@
       <origin
         xyz="0 0 0"
-        rpy="0 0 0" />
+        rpy="-1.57079632649567 1.57079632649567 -1.57079632649567" />
       <geometry>
         <mesh
@@ -445,5 +472,5 @@
       <origin
         xyz="0 0 0"
-        rpy="0 0 0" />
+        rpy="1.57 0 0" />
       <geometry>
         <mesh
@@ -453,18 +480,18 @@
   </link>
   <joint
-    name="komodo_$(arg komodo_id)_Front_Camera_joint"
+    name="Front_Camera_joint"
     type="fixed">
     <origin
       xyz="0.262250027816762 0.0875000000000051 0.100000000000001"
-      rpy="-1.57079632679489 -6.93084604642783E-17 -1.5707963267949" />
-    <parent
-      link="komodo_$(arg komodo_id)_base_link" />
-    <child
-      link="komodo_$(arg komodo_id)_Front_Camera_link" />
+      rpy="0 0 0" />
+    <parent
+      link="base_link" />
+    <child
+      link="Front_Camera_link" />
     <axis
       xyz="0 0 1" />
   </joint>
   <link
-    name="komodo_$(arg komodo_id)_Laser_link">
+    name="Laser_link">
     <inertial>
       <origin
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
File: ric/ric_description/lizi/lizi.xacro (robot description, xacro)
@@ -1,7 +1,25 @@
 <?xml version="1.0"?>
 <robot xmlns:xacro="http://www.ros.org/wiki/lizi_robot" name="lizi_urdf">
-<xacro:property name="lizi_color" value="0 0.517 0.26 1" />
-  <link
-    name="lizi_$(arg lizi_id)_base_link">
+<xacro:property name="lizi_color" value="0.0 0.0 0.0 1" />
+<!-- Dummy inertia link & Joint -->
+  <link
+    name="dummy_link">
+</link>
+  <joint
+    name="dummy_joint"
+    type="fixed">
+    <origin
+      xyz="0.0 0.0 0.0"
+      rpy="0 0 0" />
+    <parent
+      link="dummy_link" />
+    <child
+      link="base_link" />
+    <axis
+      xyz="0 0 0" />
+  </joint>
+<!-- Dummy link & node -->
+  <link
+    name="base_link">
     <inertial>
       <origin
@@ -43,5 +61,5 @@
   </link>
   <link
-    name="lizi_$(arg lizi_id)_FL_Wheel_link">
+    name="FL_Wheel_link">
     <inertial>
       <origin
@@ -61,5 +79,5 @@
       <origin
         xyz="0 0 0"
-        rpy="0 0 0" />
+        rpy="3.14159265359 0 0" />
       <geometry>
         <mesh
@@ -75,26 +93,28 @@
       <origin
         xyz="0 0 0"
-        rpy="0 0 0" />
-      <geometry>
-        <mesh
-          filename="package://ric_description/lizi/meshes/FL_Wheel_Link.STL" />
-      </geometry>
-    </collision>
-  </link>
-  <joint
-    name="lizi_$(arg lizi_id)_FL_Wheel_Joint"
+        rpy="1.5707963267949 0 0" />
+      <geometry>
+        <!--mesh
+          filename="package://ric_description/lizi/meshes/FL_Wheel_Link.STL" /-->
+        <cylinder length="0.02" radius="0.068"
+          />
+      </geometry>
+    </collision>
+  </link>
+  <joint
+    name="FL_Wheel_Joint"
     type="continuous">
     <origin
       xyz="0.118 0.1338 0.026"
-      rpy="0 0 -1.3371E-16" />
-    <parent
-      link="lizi_$(arg lizi_id)_base_link" />
-    <child
-      link="lizi_$(arg lizi_id)_FL_Wheel_link" />
+      rpy="3.14159265359 0 -1.3371E-16" />
+    <parent
+      link="base_link" />
+    <child
+      link="FL_Wheel_link" />
     <axis
       xyz="0 -1 0" />
   </joint>
   <link
-    name="lizi_$(arg lizi_id)_RL_Wheel_link">
+    name="RL_Wheel_link">
     <inertial>
       <origin
@@ -114,5 +134,5 @@
       <origin
         xyz="0 0 0"
-        rpy="0 0 0" />
+        rpy="3.14159265359 0 0" />
       <geometry>
         <mesh
@@ -128,21 +148,23 @@
       <origin
         xyz="0 0 0"
-        rpy="0 0 0" />
-      <geometry>
-        <mesh
-          filename="package://ric_description/lizi/meshes/RL_Wheel_Link.STL" />
-      </geometry>
-    </collision>
-  </link>
-  <joint
-    name="lizi_$(arg lizi_id)_RL_Wheel_Joint"
+        rpy="1.5707963267949 0 0" />
+      <geometry>
+        <!--mesh
+          filename="package://ric_description/lizi/meshes/RL_Wheel_Link.STL" /-->
+<cylinder length="0.02" radius="0.068"
+          />
+      </geometry>
+    </collision>
+  </link>
+  <joint
+    name="RL_Wheel_Joint"
     type="continuous">
     <origin
       xyz="-0.118 0.1338 0.026"
-      rpy="0 0 -6.6853E-16" />
-    <parent
-      link="lizi_$(arg lizi_id)_base_link" />
-    <child
-      link="lizi_$(arg lizi_id)_RL_Wheel_link" />
+      rpy="3.14159265359 0 -6.6853E-16" />
+    <parent
+      link="base_link" />
+    <child
+      link="RL_Wheel_link" />
     <axis
       xyz="0 -1 0" />
@@ -152,5 +174,5 @@
   </joint>
   <link
-    name="lizi_$(arg lizi_id)_RR_Wheel_link">
+    name="RR_Wheel_link">
     <inertial>
       <origin
@@ -184,13 +206,15 @@
       <origin
         xyz="0 0 0"
-        rpy="0 0 0" />
-      <geometry>
-        <mesh
-          filename="package://ric_description/lizi/meshes/RR_Wheel_Link.STL" />
-      </geometry>
-    </collision>
-  </link>
-  <joint
-    name="lizi_$(arg lizi_id)_RR_Wheel_Joint"
+        rpy="1.5707963267949 0 0" />
+      <geometry>
+        <!--mesh
+          filename="package://ric_description/lizi/meshes/RR_Wheel_Link.STL" /-->
+<cylinder length="0.02" radius="0.068"
+          />
+      </geometry>
+    </collision>
+  </link>
+  <joint
+    name="RR_Wheel_Joint"
     type="continuous">
     <origin
@@ -198,12 +222,12 @@
       rpy="-1.2938E-16 -1.2938E-15 -6.6853E-16" />
     <parent
-      link="lizi_$(arg lizi_id)_base_link" />
-    <child
-      link="lizi_$(arg lizi_id)_RR_Wheel_link" />
+      link="base_link" />
+    <child
+      link="RR_Wheel_link" />
     <axis
       xyz="0 1 0" />
   </joint>
   <link
-    name="lizi_$(arg lizi_id)_FR_Wheel_link">
+    name="FR_Wheel_link">
     <inertial>
       <origin
@@ -237,13 +261,14 @@
       <origin
         xyz="0 0 0"
-        rpy="0 0 0" />
-      <geometry>
-        <mesh
-          filename="package://ric_description/lizi/meshes/FR_Wheel_Link.STL" />
-      </geometry>
-    </collision>
-  </link>
-  <joint
-    name="lizi_$(arg lizi_id)_FR_Wheel_Joint"
+        rpy="1.5707963267949 0 0" />
+      <geometry>
+        <!--mesh
+          filename="package://ric_description/lizi/meshes/FR_Wheel_Link.STL" /-->
+<cylinder length="0.02" radius="0.068"/>
+      </geometry>
+    </collision>
+  </link>
+  <joint
+    name="FR_Wheel_Joint"
     type="continuous">
     <origin
@@ -251,12 +276,12 @@
       rpy="4.4216E-16 -0.0061583 -2.6824E-16" />
     <parent
-      link="lizi_$(arg lizi_id)_base_link" />
-    <child
-      link="lizi_$(arg lizi_id)_FR_Wheel_link" />
+      link="base_link" />
+    <child
+      link="FR_Wheel_link" />
     <axis
       xyz="0 1 0" />
   </joint>
   <link
-    name="lizi_$(arg lizi_id)_Asus_Pan_link">
+    name="Asus_Pan_link">
     <inertial>
       <origin
@@ -298,5 +323,5 @@
   </link>
   <joint
-    name="lizi_$(arg lizi_id)_Asus_Pan_Joint"
+    name="Asus_Pan_Joint"
     type="revolute">
     <origin
@@ -304,15 +329,17 @@
       rpy="2.1253E-16 8.5011E-16 0" />
     <parent
-      link="lizi_$(arg lizi_id)_base_link" />
-    <child
-      link="lizi_$(arg lizi_id)_Asus_Pan_link" />
+      link="base_link" />
+    <child
+      link="Asus_Pan_link" />
     <axis
       xyz="0 0 -1" />
     <limit
-      effort="0"
+      lower="-1"
+      upper="1"
+      effort="10"
       velocity="0" />
   </joint>
   <link
-    name="lizi_$(arg lizi_id)_Asus_Camera_link">
+    name="Asus_Camera_link">
     <inertial>
       <origin
@@ -346,5 +373,5 @@
       <origin
         xyz="0 0 0"
-        rpy="0 0 0" />
+        rpy="1.5707963267949 0 0" />
       <geometry>
         <mesh
@@ -354,5 +381,5 @@
   </link>
   <joint
-    name="lizi_$(arg lizi_id)_Asus_Tilt_Joint"
+    name="Asus_Tilt_Joint"
     type="revolute">
     <origin
@@ -360,15 +387,17 @@
       rpy="0 0 0" />
     <parent
-      link="lizi_$(arg lizi_id)_Asus_Pan_link" />
-    <child
-      link="lizi_$(arg lizi_id)_Asus_Camera_link" />
+      link="Asus_Pan_link" />
+    <child
+      link="Asus_Camera_link" />
     <axis
       xyz="0 1 0" />
     <limit
-      effort="0"
+      lower="-1"
+      upper="1"
+      effort="10"
       velocity="0" />
   </joint>
   <link
-    name="lizi_$(arg lizi_id)_Right_URF_link">
+    name="Right_URF_link">
     <inertial>
       <origin
@@ -410,5 +439,5 @@
   </link>
   <joint
-    name="lizi_$(arg lizi_id)_Right_URF_Joint"
+    name="Right_URF_Joint"
     type="fixed">
     <origin
@@ -416,12 +445,12 @@
       rpy="0 2.6072E-16 -1.57" />
     <parent
-      link="lizi_$(arg lizi_id)_base_link" />
-    <child
-      link="lizi_$(arg lizi_id)_Right_URF_link" />
+      link="base_link" />
+    <child
+      link="Right_URF_link" />
     <axis
       xyz="0 0 0" />
   </joint>
   <link
-    name="lizi_$(arg lizi_id)_Left_URF_link">
+    name="Left_URF_link">
     <inertial>
       <origin
@@ -463,5 +492,5 @@
   </link>
   <joint
-    name="lizi_$(arg lizi_id)_Left_URF_Joint"
+    name="Left_URF_Joint"
     type="fixed">
     <origin
@@ -469,12 +498,12 @@
       rpy="0 0 1.57" />
     <parent
-      link="lizi_$(arg lizi_id)_base_link" />
-    <child
-      link="lizi_$(arg lizi_id)_Left_URF_link" />
+      link="base_link" />
+    <child
+      link="Left_URF_link" />
     <axis
       xyz="0 0 0" />
   </joint>
   <link
-    name="lizi_$(arg lizi_id)_Rear_URF_link">
+    name="Rear_URF_link">
     <inertial>
       <origin
@@ -516,5 +545,5 @@
   </link>
   <joint
-    name="lizi_$(arg lizi_id)_Rear_URF_Joint"
+    name="Rear_URF_Joint"
     type="fixed">
     <origin
@@ -522,12 +551,12 @@
       rpy="0 0 3.14" />
     <parent
-      link="lizi_$(arg lizi_id)_base_link" />
-    <child
-      link="lizi_$(arg lizi_id)_Rear_URF_link" />
+      link="base_link" />
+    <child
+      link="Rear_URF_link" />
     <axis
       xyz="0 0 0" />
   </joint>
   <link
-    name="lizi_$(arg lizi_id)_Laser_link">
+    name="Laser_link">
     <inertial>
       <origin
@@ -569,5 +598,5 @@
   </link>
   <joint
-    name="lizi_$(arg lizi_id)_Laser_Joint"
+    name="Laser_Joint"
     type="fixed">
     <origin
@@ -575,12 +604,12 @@
       rpy="2.1253E-16 8.5011E-16 -2.6741E-16" />
     <parent
-      link="lizi_$(arg lizi_id)_base_link" />
-    <child
-      link="lizi_$(arg lizi_id)_Laser_link" />
+      link="base_link" />
+    <child
+      link="Laser_link" />
     <axis
       xyz="0 0 0" />
   </joint>
   <link
-    name="lizi_$(arg lizi_id)_Camera_link">
+    name="Camera_link">
     <inertial>
       <origin
@@ -622,5 +651,5 @@
   </link>
   <joint
-    name="lizi_$(arg lizi_id)_Camera_Joint"
+    name="Camera_Joint"
     type="fixed">
     <origin
@@ -628,9 +657,304 @@
       rpy="1.6519E-18 -0.0061583 -2.6824E-16" />
     <parent
-      link="lizi_$(arg lizi_id)_base_link" />
-    <child
-      link="lizi_$(arg lizi_id)_Camera_link" />
+      link="base_link" />
+    <child
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